File: _autosave-Southpaw-65.kicad_pcb (KiCad board)
At the start: 2 copper layers, 196 parts, among them J1 USB_C_Receptacle_USB2.0, SW1 SW_Push, U1 ATmega32A-PU, Y1 16MHz

Commit message: Arranged the switches on the PCB
Parts:
- D0-0, D1-0, D2-0, D3-0: value SOD-123 -> (none)
- moved MX3-19 719.2 mm to (430.2, 90.5)
- moved MX4-15 701.5 mm to (392.1, 109.5)
- moved MX3-15 685.0 mm to (385.0, 90.5)
- moved U1 683.9 mm to (423.1, -34.1)
- moved MX3-18 668.8 mm to (411.2, 90.5)
- moved MX3-13 631.1 mm to (339.7, 90.5)
- moved MX4-19 620.2 mm to (430.2, 109.5)
- moved MX3-14 617.6 mm to (358.8, 90.5)
- moved MX4-12 602.9 mm to (311.1, 109.5)
- moved MX3-11 572.1 mm to (301.6, 90.5)
- moved MX4-13 551.8 mm to (351.6, 109.5)
- moved MX4-14 543.3 mm to (373.1, 109.5)
- moved MX4-10 530.2 mm to (273.1, 109.5)
- moved MX4-18 529.7 mm to (411.2, 109.5)
- moved MX3-9 503.4 mm to (263.5, 90.5)
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