File: Southpaw-65.kicad_pcb (KiCad board)
At the start: 2 copper layers, 196 parts, among them J1 USB_C_Receptacle_USB2.0, SW1 SW_Push, U1 ATmega32A-PU, Y1 16MHz

Commit message: Backup #3
Parts:
- D0-0, D1-0, D2-0, D3-0: value SOD-123 -> (none)
- moved MX3-19 719.2 mm to (430.2, 90.5)
- moved MX4-15 701.5 mm to (392.1, 109.5)
- moved MX3-15 685.0 mm to (385.0, 90.5)
- moved U1 683.9 mm to (423.1, -34.1)
- moved MX3-18 668.8 mm to (411.2, 90.5)
- moved MX3-13 631.1 mm to (339.7, 90.5)
- moved MX4-19 620.2 mm to (430.2, 109.5)
- moved MX3-14 617.6 mm to (358.8, 90.5)
- moved MX4-12 602.9 mm to (311.1, 109.5)
- moved MX3-11 572.1 mm to (301.6, 90.5)
- moved MX4-13 551.8 mm to (351.6, 109.5)
- moved MX4-14 543.3 mm to (373.1, 109.5)
- moved MX4-10 530.2 mm to (273.1, 109.5)
- moved MX4-18 529.7 mm to (411.2, 109.5)
- moved MX3-9 503.4 mm to (263.5, 90.5)
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
Commit message: Backup #3
Parts:
- added Y1: 16MHz, Crystal:Crystal_HC49-U_Horizontal, F.Cu at (-23.0, -8.73)
- D0-0, D1-0, D2-0, D3-0: value (none) -> SOD-123
- moved D4-10 525.0 mm to (250.8, 12.7), turned to 270 degrees
- moved D3-9 493.8 mm to (235.7, 9.53), turned to 270 degrees
- moved D4-8 469.9 mm to (212.7, 12.7), turned to 270 degrees
- moved D4-6 465.3 mm to (174.6, 12.7), turned to 270 degrees
- moved D4-5 447.6 mm to (155.6, 12.7), turned to 270 degrees
- moved D0-10 442.5 mm to (266.7, 0.00), turned to 270 degrees
- moved D4-3 434.2 mm to (106.4, 12.7), turned to 270 degrees
- moved D2-11 418.7 mm to (277.8, 6.35), turned to 270 degrees
- moved D4-2 418.4 mm to (87.3, 12.7), turned to 270 degrees
- moved D3-11 409.0 mm to (273.8, 9.53), turned to 270 degrees
- moved D2-10 402.6 mm to (258.8, 6.35), turned to 270 degrees
- moved D0-9 398.4 mm to (247.7, 0.00), turned to 270 degrees
- moved D2-8 394.5 mm to (220.7, 6.35), turned to 270 degrees
- moved D0-7 393.6 mm to (209.6, 0.00), turned to 270 degrees
- moved D3-10 390.3 mm to (254.8, 9.53), turned to 270 degrees
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Connections:
- C1 pad 1: C17 -> C16
- C3 pad 1: C16 -> C17
- D1-10 pad 1: Net-(D1-10-Pad1) -> ROW1
- D1-11 pad 1: Net-(D1-10-Pad1) -> ROW1
- D1-12 pad 1: Net-(D1-10-Pad1) -> ROW1
- D1-13 pad 1: Net-(D1-10-Pad1) -> ROW1
- D1-14 pad 1: Net-(D1-10-Pad1) -> ROW1
- D1-15 pad 1: Net-(D1-10-Pad1) -> ROW1
- D1-16 pad 1: Net-(D1-10-Pad1) -> ROW1
- D1-18 pad 1: Net-(D1-10-Pad1) -> ROW1
- D1-19 pad 1: Net-(D1-10-Pad1) -> ROW1
- D1-7 pad 1: Net-(D1-10-Pad1) -> ROW1
- D1-8 pad 1: Net-(D1-10-Pad1) -> ROW1
- D1-9 pad 1: Net-(D1-10-Pad1) -> ROW1
- D2-10 pad 1: Net-(D2-10-Pad1) -> ROW2
- D2-11 pad 1: Net-(D2-10-Pad1) -> ROW2
- D2-12 pad 1: Net-(D2-10-Pad1) -> ROW2
- D2-13 pad 1: Net-(D2-10-Pad1) -> ROW2
- D2-14 pad 1: Net-(D2-10-Pad1) -> ROW2
- D2-15 pad 1: Net-(D2-10-Pad1) -> ROW2
- D2-18 pad 1: Net-(D2-10-Pad1) -> ROW2
- D2-19 pad 1: Net-(D2-10-Pad1) -> ROW2
- D2-7 pad 1: Net-(D2-10-Pad1) -> ROW2
- D2-8 pad 1: Net-(D2-10-Pad1) -> ROW2
- D2-9 pad 1: Net-(D2-10-Pad1) -> ROW2
- MX1-11 pad 1: Net-(MX1-11-Pad1) -> COL11
- MX1-15 pad 1: Net-(MX1-15-Pad1) -> COL15
- MX1-4 pad 1: Net-(MX1-4-Pad1) -> COL4
- MX1-7 pad 1: Net-(MX1-7-Pad1) -> COL7
- MX2-11 pad 1: Net-(MX1-11-Pad1) -> COL11
- MX2-15 pad 1: Net-(MX1-15-Pad1) -> COL15
- MX2-4 pad 1: Net-(MX1-4-Pad1) -> COL4
- MX2-7 pad 1: Net-(MX1-7-Pad1) -> COL7
- MX3-11 pad 1: Net-(MX1-11-Pad1) -> COL11
- MX3-15 pad 1: Net-(MX1-15-Pad1) -> COL15
- MX3-4 pad 1: Net-(MX1-4-Pad1) -> COL4
- MX3-7 pad 1: Net-(MX1-7-Pad1) -> COL7
- MX4-14 pad 1: Net-(MX4-14-Pad1) -> COL14
- MX4-15 pad 1: Net-(MX1-15-Pad1) -> COL15
- MX4-4 pad 1: Net-(MX1-4-Pad1) -> COL4

Commit message: Started tracing and working on pathing
Parts:
- moved SW1 811.9 mm to (538.2, 89.8)
- moved D0-16 794.4 mm to (515.1, 88.9), turned to 270 degrees
- moved D3-14 747.9 mm to (445.3, 86.0), turned to 270 degrees
- moved D0-14 734.3 mm to (433.4, 95.6), turned to 270 degrees
- moved D0-15 730.9 mm to (452.4, 95.6), turned to 270 degrees
- moved D4-14 718.8 mm to (449.3, 82.9), turned to 270 degrees
- moved D3-13 717.5 mm to (426.2, 86.0), turned to 270 degrees
- moved D3-19 700.7 mm to (502.4, 86.0), turned to 270 degrees
- moved D4-13 699.7 mm to (430.2, 82.9), turned to 270 degrees
- moved D3-12 699.3 mm to (407.2, 86.0), turned to 270 degrees
- moved D4-12 692.0 mm to (411.2, 82.9), turned to 270 degrees
- moved D3-18 681.6 mm to (483.4, 86.0), turned to 270 degrees
- moved D4-15 609.0 mm to (468.3, 82.9), turned to 270 degrees
- moved D3-15 600.5 mm to (464.3, 86.0), turned to 270 degrees
- moved D4-19 580.1 mm to (506.4, 82.9), turned to 270 degrees
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Connections:
- MX0-7 pad 2: Net-(MX0-7-Pad2) -> Net-(D0-7-Pad2)
- MX1-0 pad 1: Net-(MX1-0-Pad1) -> COL0
- MX2-0 pad 1: Net-(MX1-0-Pad1) -> COL0
- MX3-0 pad 1: Net-(MX1-0-Pad1) -> COL0
- MX4-0 pad 1: Net-(MX1-0-Pad1) -> COL0
Routing:
- net GND: track 0.00 -> 545.2 mm, vias 0 -> 7
- net ROW0: track 0.00 -> 432.0 mm
- net Reset: track 0.00 -> 418.8 mm
- net ROW1: track 0.00 -> 395.4 mm
- net ROW2: track 0.00 -> 376.0 mm
- net ROW4: track 0.00 -> 375.8 mm
- net ROW3: track 0.00 -> 375.7 mm
- net +5V: track 0.00 -> 149.3 mm, vias 0 -> 3
- net Net-(D4-18-Pad2): track 0.00 -> 141.6 mm
- net Net-(D4-19-Pad2): track 0.00 -> 136.9 mm
- net Net-(D4-5-Pad2): track 0.00 -> 128.9 mm
- net Net-(D4-6-Pad2): track 0.00 -> 127.5 mm
- net Net-(D4-14-Pad2): track 0.00 -> 126.1 mm
- net Net-(D4-15-Pad2): track 0.00 -> 124.4 mm
- net Net-(D4-8-Pad2): track 0.00 -> 124.2 mm
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Other:
- board outline added: 452.4 x 139.7 mm
- net class Default: trace_width 0.25 -> 0.254
- net class Power added: clearance 0.2, trace_width 0.381, via_dia 0.8, via_drill 0.4

Commit message: Finished all tracks
Connections:
- net Net-(U1-Pad18) renamed REA
- net Net-(U1-Pad19) renamed REB
- MX1-18 pad 1: Net-(MX1-18-Pad1) -> COL18
- MX2-18 pad 1: Net-(MX1-18-Pad1) -> COL18
- MX3-18 pad 1: Net-(MX1-18-Pad1) -> COL18
- MX4-18 pad 1: Net-(MX1-18-Pad1) -> COL18
Routing:
- net COL11: track 0.00 -> 569.0 mm, vias 0 -> 2
- net COL17: track 0.00 -> 524.2 mm, vias 0 -> 3
- net COL18: track 0.00 -> 516.5 mm, vias 0 -> 4
- net COL15: track 0.00 -> 512.0 mm, vias 0 -> 3
- net COL14: track 0.00 -> 491.3 mm, vias 0 -> 3
- net COL16: track 0.00 -> 490.7 mm, vias 0 -> 9
- net COL19: track 0.00 -> 472.8 mm, vias 0 -> 3
- net COL13: track 0.00 -> 464.4 mm, vias 0 -> 3
- net COL12: track 0.00 -> 409.8 mm, vias 0 -> 3
- net COL10: track 0.00 -> 310.3 mm, vias 0 -> 3
- net COL9: track 0.00 -> 289.4 mm, vias 0 -> 3
- net COL8: track 0.00 -> 264.8 mm, vias 0 -> 3
- net COL7: track 0.00 -> 242.9 mm, vias 0 -> 3
- net COL1: track 0.00 -> 214.2 mm, vias 0 -> 5
- net COL6: track 0.00 -> 212.7 mm, vias 0 -> 3
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Other:
- board size 452.4 x 139.7 mm -> 452.4 x 139.4 mm

Commit message: Added mounting holes to pcb added changed dimensions of PCB
Parts:
- added H1: MountingHole, MountingHole:MountingHole_3.2mm_M3, F.Cu at (109.6, 87.5)
- added H2: MountingHole, MountingHole:MountingHole_3.2mm_M3, F.Cu at (197.6, 102.6)
- added H3: MountingHole, MountingHole:MountingHole_3.2mm_M3, F.Cu at (549.9, 87.5)
- added H4: MountingHole, MountingHole:MountingHole_3.2mm_M3, F.Cu at (232.9, 102.6)
- added H5: MountingHole, MountingHole:MountingHole_3.2mm_M3, F.Cu at (109.6, 206.1)
- added H6: MountingHole, MountingHole:MountingHole_3.2mm_M3, F.Cu at (197.6, 211.3)
- added H7: MountingHole, MountingHole:MountingHole_3.2mm_M3, F.Cu at (549.9, 206.1)
- added H8: MountingHole, MountingHole:MountingHole_3.2mm_M3, F.Cu at (232.9, 211.3)
- moved SW1 4.00 mm to (534.2, 89.8)
- moved J1 2.51 mm to (218.3, 82.4)
Routing:
- net COL11: track 569.0 -> 408.5 mm
- net (no net): track 43.0 -> 0.00 mm, vias 1 -> 0
- net Net-(D1-19-Pad2): track 78.8 -> 86.7 mm, vias 0 -> 4
- net GND: track 594.6 -> 589.5 mm
- net Net-(J1-PadB5): track 169.4 -> 165.4 mm, vias 2 -> 0
- net ROW4: track 506.0 -> 510.0 mm, vias 1 -> 3
- net Reset: track 464.3 -> 460.3 mm
- net Net-(J1-PadA5): track 194.6 -> 194.5 mm, vias 6 -> 5
Other:
- board size 452.4 x 139.4 mm -> 457.2 x 139.7 mm

Commit message: Redoing Board
Parts:
- removed the Y1 at (213.4, 129.4)
- removed the Y1 at (213.4, 117.5)
- added Y1: 16MHz, Crystal:Crystal_HC49-U_Horizontal, F.Cu at (140.2, -184.3)
- moved MX4-19 499.8 mm to (222.4, -196.6)
- moved H7 492.5 mm to (156.2, -89.7)
- moved MX3-15 490.9 mm to (108.8, -134.7)
- moved MX4-18 485.7 mm to (178.4, -155.5)
- moved MX4-15 478.3 mm to (131.4, -114.5)
- moved MX3-19 477.7 mm to (171.8, -135.3)
- moved SW1 475.3 mm to (130.7, -161.3)
- moved MX4-14 474.0 mm to (101.7, -94.3)
- moved MX2-18 471.5 mm to (190.3, -196.6)
- moved MX4-10 465.1 mm to (158.8, -217.4)
- moved MX1-18 453.0 mm to (183.1, -175.7)
- moved MX3-18 450.6 mm to (233.1, -176.4)
- moved MX4-8 446.9 mm to (120.7, -196.6)
- moved MX4-12 440.5 mm to (255.2, -217.4)
- moved MX4-13 440.1 mm to (296.9, -217.4)
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Routing:
- net ROW0: track 601.9 -> 0.00 mm, vias 3 -> 0
- net GND: track 589.5 -> 0.00 mm, vias 11 -> 0
- net ROW1: track 554.7 -> 0.00 mm, vias 3 -> 0
- net ROW2: track 527.7 -> 0.00 mm, vias 1 -> 0
- net COL17: track 524.2 -> 0.00 mm, vias 3 -> 0
- net ROW3: track 516.8 -> 0.00 mm, vias 1 -> 0
- net COL18: track 516.5 -> 0.00 mm, vias 4 -> 0
- net COL15: track 512.0 -> 0.00 mm, vias 3 -> 0
- net ROW4: track 510.0 -> 0.00 mm, vias 3 -> 0
- net COL14: track 491.3 -> 0.00 mm, vias 3 -> 0
- net COL16: track 490.7 -> 0.00 mm, vias 9 -> 0
- net COL19: track 472.8 -> 0.00 mm, vias 3 -> 0
- net COL13: track 464.4 -> 0.00 mm, vias 3 -> 0
- net Reset: track 460.3 -> 0.00 mm, vias 3 -> 0
- net COL12: track 409.8 -> 0.00 mm, vias 3 -> 0
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Other:
- board outline removed

Commit message: Made the switch matrix in the pcb
Parts:
- moved MX4-19 447.4 mm to (485.8, 165.1)
- moved MX3-15 434.6 mm to (440.5, 146.1)
- moved MX4-18 431.2 mm to (466.7, 165.1)
- moved MX4-15 422.1 mm to (447.7, 165.1)
- moved MX3-19 421.6 mm to (485.8, 146.1)
- moved MX4-10 418.5 mm to (328.6, 165.1)
- moved MX2-18 417.9 mm to (454.8, 127.0)
- moved MX4-14 417.3 mm to (428.6, 165.1)
- moved MX4-8 399.5 mm to (290.5, 165.1)
- moved MX4-12 398.4 mm to (366.7, 165.1)
- moved MX3-18 398.2 mm to (466.7, 146.1)
- moved MX4-13 398.1 mm to (407.2, 165.1)
- moved MX1-18 397.8 mm to (462.0, 108.0)
- moved MX0-19 374.4 mm to (485.8, 88.9)
- moved MX4-5 368.3 mm to (228.6, 165.1)
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
Commit message: Added some diodes into matrix
Parts:
- moved D3-2 325.5 mm to (131.0, 47.6), turned to 270 degrees
- moved D2-2 322.7 mm to (127.0, 52.4), turned to 270 degrees
- moved U1 310.6 mm to (164.1, 105.7)
- moved D1-2 215.0 mm to (123.0, 57.1), turned to 270 degrees
- moved J1 208.3 mm to (169.6, 40.1)
- moved D4-2 192.1 mm to (134.9, 42.9), turned to 270 degrees
- moved C8 170.7 mm to (168.7, 88.9)
- moved D0-2 35.2 mm to (119.1, 61.9), turned to 270 degrees
- moved D1-0 7.94 mm to (84.9, 57.1), turned to 270 degrees
- moved D1-1 7.94 mm to (104.0, 57.1), turned to 270 degrees
- moved D2-0 7.94 mm to (88.9, 52.4), turned to 270 degrees
- moved D2-1 7.94 mm to (108.0, 52.4), turned to 270 degrees
- moved D3-0 7.94 mm to (92.9, 47.6), turned to 270 degrees
- moved D3-1 7.94 mm to (111.9, 47.6), turned to 270 degrees
- moved D4-0 7.94 mm to (96.8, 42.9), turned to 270 degrees
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Routing:
- net Net-(D4-1-Pad2): track 0.00 -> 118.3 mm
- net Net-(D4-0-Pad2): track 0.00 -> 118.3 mm
- net COL2: track 0.00 -> 113.9 mm
- net COL3: track 0.00 -> 97.2 mm
- net COL0: track 0.00 -> 96.4 mm
- net Net-(D3-0-Pad2): track 0.00 -> 95.9 mm
- net Net-(D3-1-Pad2): track 0.00 -> 95.9 mm
- net COL1: track 0.00 -> 94.8 mm
- net Net-(D2-1-Pad2): track 0.00 -> 75.0 mm
- net Net-(D2-0-Pad2): track 0.00 -> 75.0 mm
- net Net-(D1-0-Pad2): track 0.00 -> 54.0 mm
- net Net-(D1-1-Pad2): track 0.00 -> 54.0 mm
- net ROW4: track 0.00 -> 38.1 mm
- net ROW3: track 0.00 -> 38.1 mm
- net ROW2: track 0.00 -> 38.1 mm
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