File: Southpaw-65.kicad_pcb (KiCad board)
At the start: 2 copper layers, 205 parts, among them J1 USB_C_Receptacle_USB2.0, SW1 SW_Push, U1 ATmega32A-PU, Y1 16MHz

Commit message: More wiring
Connections:
- U1 pad 1: Net-(U1-Pad1) -> COL3
- U1 pad 14: Net-(U1-Pad14) -> ROW4
- U1 pad 2: Net-(U1-Pad2) -> COL2
- U1 pad 3: Net-(U1-Pad3) -> COL1
- U1 pad 39: Net-(U1-Pad39) -> COL4
- U1 pad 4: Net-(U1-Pad4) -> COL0
- U1 pad 40: Net-(U1-Pad40) -> COL5
- U1 pad 5: Net-(U1-Pad5) -> ROW0
- U1 pad 6: Net-(U1-Pad6) -> ROW1
- U1 pad 7: Net-(U1-Pad7) -> ROW2
- U1 pad 8: Net-(U1-Pad8) -> ROW3
Routing:
- net COL19: track 105.2 -> 480.3 mm, vias 0 -> 1
- net COL18: track 126.2 -> 477.1 mm, vias 2 -> 3
- net COL17: track 123.1 -> 452.6 mm
- net COL16: track 119.5 -> 395.3 mm
- net ROW3: track 375.6 -> 647.9 mm, vias 2 -> 4
- net ROW4: track 380.1 -> 651.4 mm, vias 3 -> 5
- net ROW2: track 389.6 -> 652.6 mm, vias 1 -> 3
- net COL15: track 135.4 -> 394.4 mm
- net ROW1: track 390.1 -> 644.1 mm, vias 0 -> 2
- net ROW0: track 409.0 -> 654.6 mm, vias 1 -> 5
- net COL14: track 135.8 -> 375.1 mm
- net COL13: track 133.9 -> 350.9 mm
- net COL12: track 132.9 -> 308.7 mm
- net COL11: track 131.4 -> 283.3 mm
- net COL0: track 96.4 -> 234.5 mm, vias 0 -> 1
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
Commit message: Lots of wiring to MCU done
Considering redoing it because thicc bottom
Parts:
- moved H5 433.6 mm to (500.1, 191.3)
- moved H7 365.8 mm to (500.1, 34.9)
- moved H3 360.7 mm to (162.7, 34.9)
- moved H2 340.2 mm to (184.2, 34.9)
- moved H8 298.8 mm to (71.4, 191.3)
- moved H6 292.7 mm to (71.4, 34.9)
- moved H1 277.7 mm to (184.2, 191.3)
- moved H4 187.4 mm to (162.7, 191.3)
Connections:
- U1 pad 15: Net-(U1-Pad15) -> COL18
- U1 pad 20: Net-(U1-Pad20) -> COL19
- U1 pad 24: Net-(U1-Pad24) -> COL15
- U1 pad 25: Net-(U1-Pad25) -> COL16
- U1 pad 27: Net-(U1-Pad27) -> COL17
- U1 pad 28: Net-(U1-Pad28) -> COL6
- U1 pad 29: Net-(U1-Pad29) -> COL7
- U1 pad 32: Net-(U1-Pad32) -> COL8
- U1 pad 33: Net-(U1-Pad33) -> COL9
- U1 pad 34: Net-(U1-Pad34) -> COL10
- U1 pad 35: Net-(U1-Pad35) -> COL11
- U1 pad 36: Net-(U1-Pad36) -> COL12
- U1 pad 37: Net-(U1-Pad37) -> COL13
- U1 pad 38: Net-(U1-Pad38) -> COL14
Routing:
- net COL14: track 375.1 -> 451.6 mm, vias 0 -> 1
- net COL13: track 350.9 -> 422.6 mm, vias 0 -> 1
- net COL12: track 308.7 -> 375.5 mm, vias 0 -> 1
- net COL11: track 283.3 -> 345.5 mm, vias 0 -> 1
- net COL10: track 269.1 -> 325.8 mm, vias 0 -> 1
- net COL9: track 242.8 -> 294.7 mm, vias 0 -> 1
- net COL16: track 395.3 -> 444.2 mm, vias 2 -> 3
- net COL8: track 229.3 -> 276.8 mm, vias 0 -> 1
- net COL15: track 394.4 -> 438.5 mm, vias 0 -> 1
- net COL7: track 203.9 -> 241.8 mm, vias 0 -> 1
- net COL19: track 480.3 -> 444.9 mm
- net COL6: track 187.8 -> 219.2 mm, vias 0 -> 1
- net COL18: track 477.1 -> 457.5 mm
- net COL17: track 452.6 -> 458.7 mm, vias 2 -> 3
- net Net-(J1-PadB8): track 5.71 -> 0.00 mm
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Other:
- board outline added: 436.2 x 164 mm

Commit message: Redid wirings
Decrease in space between pcb bottom, and switches
Parts:
- moved H8 7.19 mm to (72.2, 184.2)
- moved H4 7.14 mm to (162.7, 184.2)
- moved H5 6.40 mm to (499.3, 184.9)
- moved H1 6.35 mm to (184.2, 184.9)
- moved H6 1.12 mm to (72.2, 35.7)
- moved H7 1.12 mm to (499.3, 35.7)
Connections:
- net REA renamed Net-(U1-Pad18)
- net REB renamed Net-(U1-Pad19)
- U1 pad 15: COL18 -> COL19
- U1 pad 20: COL19 -> Net-(U1-Pad20)
- U1 pad 24: COL15 -> COL16
- U1 pad 25: COL16 -> COL17
- U1 pad 26: Net-(U1-Pad26) -> COL8
- U1 pad 27: COL17 -> COL9
- U1 pad 28: COL6 -> COL18
- U1 pad 29: COL7 -> COL10
- U1 pad 32: COL8 -> COL11
- U1 pad 33: COL9 -> COL12
- U1 pad 34: COL10 -> COL13
- U1 pad 35: COL11 -> COL15
- U1 pad 36: COL12 -> COL6
- U1 pad 37: COL13 -> COL14
- U1 pad 38: COL14 -> COL7
Routing:
- net COL4: track 202.8 -> 127.7 mm
- net COL5: track 241.2 -> 175.1 mm
- net COL6: track 219.2 -> 271.7 mm
- net COL7: track 241.8 -> 280.8 mm
- net COL8: track 276.8 -> 252.8 mm
- net COL17: track 458.7 -> 437.1 mm, vias 3 -> 5
- net COL16: track 444.2 -> 424.4 mm, vias 3 -> 5
- net COL9: track 294.7 -> 275.5 mm
- net COL14: track 451.6 -> 433.0 mm, vias 1 -> 3
- net COL10: track 325.8 -> 308.8 mm
- net COL11: track 345.5 -> 332.3 mm
- net COL13: track 422.6 -> 409.6 mm
- net COL12: track 375.5 -> 362.5 mm
- net COL15: track 438.5 -> 449.4 mm, vias 1 -> 3
- net COL18: track 457.5 -> 452.3 mm, vias 3 -> 5
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Other:
- board size 436.2 x 164 mm -> 436.2 x 158.6 mm

Commit message: Added encoders
Parts:
- removed MX3-0: MX-NoLED, MX_Alps_Hybrid:MX-1U
- added MX0-0B1: MX-NoLED, MX_Only:MXOnly-2U, F.Cu at (88.9, 117.5)
- added MX3-0A1: MX-NoLED, MX_Only:MXOnly-1U, F.Cu at (88.9, 146.1)
- added MX3-0B1: MX-NoLED, MX_Only:MXOnly-2U, F.Cu at (88.9, 155.6)
- added MX4-2B1: MX-NoLED, MX_Only:MXOnly-2U, F.Cu at (136.5, 165.1)
- added R4: 1k, Resistor_THT:R_Axial_DIN0207_L6.3mm_D2.5mm_P7.62mm_Horizontal, F.Cu at (465.1, 59.5)
- added R7: 1k, Resistor_THT:R_Axial_DIN0207_L6.3mm_D2.5mm_P7.62mm_Horizontal, F.Cu at (469.9, 59.5)
- added R8: 1k, Resistor_THT:R_Axial_DIN0207_L6.3mm_D2.5mm_P7.62mm_Horizontal, F.Cu at (465.1, 63.5)
- added R9: 1k, Resistor_THT:R_Axial_DIN0207_L6.3mm_D2.5mm_P7.62mm_Horizontal, F.Cu at (469.9, 63.5)
- added SW2: Rotary_Encoder, Rotary_Encoder:RotaryEncoder_Alps_EC11E_Vertical_H20mm, F.Cu at (478.6, 61.1)
- added SW3: Rotary_Encoder, Rotary_Encoder:RotaryEncoder_Alps_EC11E_Vertical_H20mm, F.Cu at (478.6, 46.0)
- MX0-0, MX0-1, MX0-10, MX0-11, MX0-12, MX0-13, MX0-14, MX0-15, MX0-16, MX0-17A1, MX0-18, MX0-19, MX0-2, MX0-3, MX0-4, MX0-5, MX0-6, MX0-7, MX0-8, MX0-9, MX1-1, MX1-10, MX1-11, MX1-12, MX1-13, MX1-14, MX1-15, MX1-16, MX1-19, MX1-2, MX1-3, MX1-5, MX1-6, MX1-7, MX1-8, MX1-9, MX2-0, MX2-1, MX2-10, MX2-11, MX2-12, MX2-13, MX2-14, MX2-15, MX2-19, MX2-2, MX2-3, MX2-5, MX2-6, MX2-7, MX2-8, MX2-9, MX3-1, MX3-10, MX3-11, MX3-12, MX3-13, MX3-14, MX3-18, MX3-19, MX3-2, MX3-3, MX3-5, MX3-6, MX3-7, MX3-8, MX3-9, MX4-0, MX4-1, MX4-14, MX4-15, MX4-18, MX4-19, MX4-3, MX4-5: footprint MX_Alps_Hybrid:MX-1U -> MX_Only:MXOnly-1U
- MX0-17B1: footprint MX_Alps_Hybrid:MX-2U -> MX_Only:MXOnly-2U
- MX1-0B1: renamed from MX1-0; footprint MX_Alps_Hybrid:MX-1U -> MX_Only:MXOnly-1U
- MX1-18, MX1-4, MX4-4: footprint MX_Alps_Hybrid:MX-1.5U -> MX_Only:MXOnly-1.5U
- MX2-18, MX3-4: footprint MX_Alps_Hybrid:MX-2.25U -> MX_Only:MXOnly-2.25U
- MX2-4, MX3-15: footprint MX_Alps_Hybrid:MX-1.75U -> MX_Only:MXOnly-1.75U
- MX4-10: footprint MX_Alps_Hybrid:MX-7U -> MX_Only:MXOnly-7U
- MX4-12, MX4-8: footprint MX_Alps_Hybrid:MX-3U -> MX_Only:MXOnly-3U
- MX4-13, MX4-6: footprint MX_Alps_Hybrid:MX-1.25U -> MX_Only:MXOnly-1.25U
- MX4-2A1: renamed from MX4-2; footprint MX_Alps_Hybrid:MX-1U -> MX_Only:MXOnly-1U
- moved D2-5 0.79 mm to (219.1, 52.4)
- moved D3-5 0.79 mm to (223.0, 47.6)
- moved D4-5 0.79 mm to (227.0, 42.9)
Connections:
- U1 pad 18: Net-(U1-Pad18) -> COL16
- U1 pad 24: COL16 -> Net-(U1-Pad24)
Routing:
- net RE-2A: track 0.00 -> 400.7 mm, vias 0 -> 2
- net RE-1A: track 0.00 -> 393.6 mm, vias 0 -> 2
- net RE-1B: track 0.00 -> 380.3 mm, vias 0 -> 2
- net RE-2B: track 0.00 -> 375.5 mm, vias 0 -> 2
- net Net-(D4-0-Pad2): track 118.3 -> 38.1 mm
- net Net-(D3-0-Pad2): track 95.9 -> 47.6 mm
- net Net-(D2-0-Pad2): track 75.0 -> 32.9 mm
- net GND: track 480.8 -> 515.1 mm
- net Net-(R7-Pad1): track 0.00 -> 20.4 mm
- net Net-(D1-0-Pad2): track 54.0 -> 74.2 mm
- net Net-(R4-Pad1): track 0.00 -> 19.8 mm
- net Net-(R9-Pad1): track 0.00 -> 19.7 mm
- net Net-(R8-Pad1): track 0.00 -> 17.7 mm
- net COL2: track 216.5 -> 228.2 mm, vias 1 -> 3
- net COL0: track 234.5 -> 225.7 mm
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
Commit message: Finished encoders and worked on fills
Connections:
- U1 pad 21: Net-(U1-Pad21) -> RE-1B
- U1 pad 22: Net-(U1-Pad22) -> RE-2A
- U1 pad 23: Net-(U1-Pad23) -> RE-1A
- U1 pad 24: Net-(U1-Pad24) -> RE-2B
Routing:
- net RE-2B: track 375.5 -> 390.0 mm
- net RE-1B: track 380.3 -> 394.1 mm
- net RE-2A: track 400.7 -> 413.5 mm
- net RE-1A: track 393.6 -> 405.7 mm
- net GND: track 515.1 -> 523.8 mm
- added copper zone on F.Cu, net GND

Commit message: Finishing Touches
Routing:
- net GND: vias 10 -> 11
- added copper zone on B.Cu, net GND

Commit message: Redid the outline for the keyboard to make it easier
Parts:
- removed H1, H2, H3, H4, H5, H6, H7, H8: MountingHole, MountingHole:MountingHole_3.2mm_M3
Routing:
- net GND: track 523.8 -> 570.0 mm, vias 11 -> 49
- net D-: track 90.8 -> 111.2 mm, vias 2 -> 6
- net D+: track 86.0 -> 101.1 mm, vias 0 -> 3
- net Reset: track 417.2 -> 414.6 mm, vias 4 -> 6
- removed copper zone on B.Cu, net GND
- removed copper zone on F.Cu, net GND
Other:
- board size 436.2 x 158.6 mm -> 427.2 x 149.6 mm
- board text added: "proton 65 By D3lta_M3"

Commit message: Altered bottom row layout and equalized dimensions of board
Left and right side of board were of different distances from the switches, so they were fixed to be equal. Bottom Row layout is now 1.25/12.5/1.25 rather than 1.5/1/1.25 this does not change the total layout as it is redistribution of space between the three keys.
Parts:
- MX4-4: footprint MX_Only:MXOnly-1.5U -> MX_Only:MXOnly-1.25U
- MX4-5: footprint MX_Only:MXOnly-1U -> MX_Only:MXOnly-1.25U
- moved MX4-4 2.38 mm to (202.4, 165.1)
- moved MX4-5 2.38 mm to (226.2, 165.1)
Routing:
- net COL5: track 175.1 -> 170.7 mm
- net COL4: track 127.7 -> 124.5 mm
- net Net-(D4-4-Pad2): track 127.0 -> 129.0 mm
- net Net-(D4-5-Pad2): track 145.1 -> 147.1 mm
Other:
- board size 427.2 x 149.6 mm -> 428.6 x 149.2 mm
